Commit message: update

File: src/my_robot_description/urdf/my_robot.urdf.xacro (robot description, xacro)
@@ -2,6 +2,8 @@
 <robot name="my_robot" xmlns:xacro="http://www.ros.org/wiki/xacro">
     <xacro:include filename="common_properties.xacro" />
-    <xacro:include filename="simple_robot_car.urdf.xacro"/>
+    <!-- <xacro:include filename="simple_robot_car.urdf.xacro"/> -->
+    <xacro:include filename="vacuum_robot_base.xacro"/>
     <xacro:include filename="simple_robot_car_gazebo.urdf.xacro"/>
-    <xacro:include filename="camera.xacro"/>
+    <!-- <xacro:include filename="camera.xacro"/> -->
+    <xacro:include filename="lidar.xacro"/>
 </robot>

File: src/my_robot_description/urdf/simple_robot_car.urdf.xacro (robot description, xacro)
@@ -1,9 +1,9 @@
 <?xml version="1.0"?>
 <robot xmlns:xacro="http://www.ros.org/wiki/xacro">
-    <xacro:property name="base_length" value="0.6" />
-    <xacro:property name="base_width" value="0.4" />
-    <xacro:property name="base_height" value="0.2" />
-    <xacro:property name="wheel_radius" value="0.1" />
-    <xacro:property name="wheel_length" value="0.05" />
+    <xacro:property name="base_length" value="0.3" />
+    <xacro:property name="base_width" value="0.3" />
+    <xacro:property name="base_height" value="0.1" />
+    <xacro:property name="wheel_radius" value="0.05" />
+    <xacro:property name="wheel_length" value="0.025" />
     <xacro:macro name="wheel_link" params="prefix">
         <link name="${prefix}_wheel_link">
@@ -24,5 +24,5 @@
         </link>
     </xacro:macro>
-    <link name="ground">
+    <link name="base_footprint">
     </link>
     <link name="base_link">
@@ -62,6 +62,6 @@
                                 xyz="0 0 0" rpy="0 0 0" />
     </link>
-    <joint name="ground_base_joint" type="fixed">
-        <parent link="ground" />
+    <joint name="base_footprint_base_joint" type="fixed">
+        <parent link="base_footprint" />
         <child link="base_link" />
         <origin xyz="0 0 ${wheel_radius}" rpy="0 0 0" />
@@ -70,5 +70,5 @@
         <parent link="base_link" />
         <child link="right_wheel_link" />
-        <origin xyz="${-base_length / 4.0} ${-base_width / 2.0 - wheel_length / 2.0} 0" rpy="0 0 0" />
+        <origin xyz="${-base_length*0 / 4.0} ${-base_width / 2.0 - wheel_length / 2.0} 0" rpy="0 0 0" />
         <axis xyz="0 1 0" />
     </joint>
@@ -76,5 +76,5 @@
         <parent link="base_link" />
         <child link="left_wheel_link" />
-        <origin xyz="${-base_length / 4.0} ${base_width / 2.0 + wheel_length / 2.0} 0" rpy="0 0 0" />
+        <origin xyz="${-base_length*0 / 4.0} ${base_width / 2.0 + wheel_length / 2.0} 0" rpy="0 0 0" />
         <axis xyz="0 1 0" />
     </joint>
